Commit message: Update tanke.common.urdf.xacro

File: rostanke_description/urdf/tanke.common.urdf.xacro (robot description, xacro)
@@ -183,5 +183,5 @@
         <axis xyz="1 0 0"/>
         <origin xyz="${plat_props['x_joint']} ${plat_props['y_joint']} ${plat_props['z_joint']}" rpy="0 0 0"/>
-        <limit lower="${lower}" upper="${uper}" effort="1.0" velocity="0.06"/>
+        <limit lower="${lower}" upper="${uper}" effort="3.0" velocity="0.6"/>
     </joint>
     <transmission name="${prefix}_transmission">
